File: Hardware/SuperButton/SuperButton.kicad_pcb (KiCad board)
At the start: 2 copper layers, 53.2 x 53.2 mm, 25 parts, among them J101 USBC, J103 EXT_LED, SW101 Switch, SW102 PROG, U101 CH552G

Commit message: Cleanup silk
Parts:
- moved J101 0.18 mm to (171.6, 67.2)
Changed lines of the file:
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@@
     (property "ki_keywords" "R resistor")
     (attr smd)
-    (fp_text reference "R102" (at 3.5075 0 90) (layer "F.SilkS")
+    (fp_text reference "R102" (at 3.5075 0 90) (layer "F.SilkS") hide
         (effects (font (size 1 1) (thickness 0.15)))
     )
-    (fp_text value "5K1" (at 0 1.65 90) (layer "F.Fab")
+    (fp_text value "5K1" (at 3.2925 -0.078572 90) (layer "F.SilkS")
         (effects (font (size 1 1) (thickness 0.15)))
     )
@@
     (property "ki_keywords" "R resistor")
     (attr smd)
-    (fp_text reference "R101" (at 3.5075 0 90) (layer "F.SilkS")
+    (fp_text reference "R101" (at 3.5075 0 90) (layer "F.SilkS") hide
         (effects (font (size 1 1) (thickness 0.15)))
     )
-    (fp_text value "5K1" (at 0 1.65 90) (layer "F.Fab")
+    (fp_text value "5K1" (at 3.2925 0.071428 90) (layer "F.SilkS")
         (effects (font (size 1 1) (thickness 0.15)))
     )
@@
   )
   (footprint "Connector_USB:USB_C_Receptacle_XKB_U262-16XN-4BVC11" (layer "F.Cu")
-    (at 171.728572 67.33 180)
+    (at 171.6 67.2 180)
     (descr "USB Type C, right-angle, SMT, https://datasheet.lcsc.com/szlcsc/1811141824_XKB-Enterprise-U262-161N-4BVC11_C319148.pdf")
     (tags "USB C Type-C Receptacle SMD")
@@
     (property "ki_keywords" "usb universal serial bus type-C USB2.0")
     (attr smd)
-    (fp_text reference "J101" (at -0.021428 0.08) (layer "F.SilkS")
+    (fp_text reference "J101" (at 0 0) (layer "F.SilkS")
         (effects (font (size 1 1) (thickness 0.15)))
     )
