File: Hardware/SuperButton/SuperButton.kicad_sch (KiCad schematic)
At the start: 0 parts

Commit message: CH552G (#3)
Parts:
- added C101, C104: 0.1uf, Capacitor_SMD:C_0805_2012Metric, symbol Device:C_Small
- added D103: STAT, LED_SMD:LED_0805_2012Metric, symbol Device:LED
- added D104: PWR, LED_SMD:LED_0805_2012Metric, symbol Device:LED
- added H101, H102, H103, H104: MountingHole, MountingHole:MountingHole_6.5mm, symbol Mechanical:MountingHole
- added J101: USBC, Connector_USB:USB_C_Receptacle_XKB_U262-16XN-4BVC11, symbol Connector:USB_C_Receptacle_USB2.0
- added J103: EXT_LED, Connector_Wire:SolderWire-0.15sqmm_1x02_P4mm_D0.5mm_OD1.5mm_Relief, symbol Connector:Conn_01x02_Socket
- added R101, R102: 5K1, Resistor_SMD:R_0805_2012Metric, symbol Device:R_Small
- added R103, R104, R105, R106: 20k, Resistor_SMD:R_0805_2012Metric, symbol Device:R_Small
- added R108: DNF, Resistor_SMD:R_0805_2012Metric, symbol Device:R_Small
- added SW101: Switch, Switch_Keyboard_Cherry_MX:SW_Cherry_MX_PCB, symbol Switch:SW_SPST
- added SW201: PROG, Button_Switch_SMD:SW_SPST_TL3342, symbol Switch:SW_Push
- added TP101: TestPoint, TestPoint:TestPoint_Pad_2.5x2.5mm, symbol Connector:TestPoint
- added U101: CH552G, Package_SO:SOP-16_3.9x9.9mm_P1.27mm, symbol KenwoodFox:CH552G
Connections:
- new net: D103.2 (A), R106.1
- new net: J103.1 (Pin_1), R108.1
- new net: R104.1, SW201.1
- new net: J101.B5 (CC2), R101.2
- new net: J101.A5 (CC1), R102.2
- new net: D104.2 (A), R103.1
- new net +3V3: C101.1, U101.16 (3V3)
- new net +5V: C104.1, J101.A4 (VBUS), J101.A9 (VBUS), J101.B4 (VBUS), J101.B9 (VBUS), J103.2 (Pin_2), R103.2, R105.2, SW201.2, U101.15 (VCC)
- new net EXT: R108.2, U101.7 (P3.1)
- new net GND: C101.2, C104.2, D103.1 (K), D104.1 (K), J101.A1 (GND), J101.A12 (GND), J101.B1 (GND), J101.B12 (GND), J101.S1 (SHIELD), R101.1, R102.1, SW101.2 (B), U101.14 (GND)
- new net RST: TP101.1, U101.6 (RST)
- new net STAT: R106.2, U101.8 (P3.0)
- new net SW_SENSE: R105.1, SW101.1 (A), U101.1 (P3.2)
- new net USB+: J101.A6 (D+), J101.B6 (D+), R104.2, U101.12 (P3.6/D+)
- new net USB-: J101.A7 (D-), J101.B7 (D-), U101.13 (P3.7/D-)
- no-connect marks 0 -> 9
Other:
- note added: "LEDs"
- note added: "MCU"
- note added: "USB"
