File: Hardware/SuperButtonX1/SuperButtonX1.kicad_pcb (KiCad board)
At the start: 2 copper layers, 53.2 x 53.2 mm, 25 parts, among them J101 USBC, J103 EXT_LED, SW101 Switch, SW102 PROG, U101 CH552G

Commit message: Clean up Super Button X1
Parts:
- moved G*** 5.37 mm to (190.4, 89.6)
- moved REF** 3.60 mm to (153.8, 96.4)
- moved REF** 3.60 mm to (153.5, 86.8)
Routing:
- net /EXT: track 41.6 -> 27.9 mm, vias 0 -> 2
- net +5V: track 90.7 -> 87.6 mm, vias 2 -> 3
- net /STAT: track 33.5 -> 33.0 mm, vias 2 -> 0
Other:
- board text added: "By FRC 1721 Tidal Force Concord, NH https://www.frc1721.org/ ${FULL_REVISION}"
- board text added: "Programmable Single Key Keyboard"
- board text removed: "Super Buttton By FRC 1721 Tidal Force https://www.frc1721.org/ ${FULL_REVISION}"
Changed lines of the file:
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@@
   )
   (footprint "1721:TIDAL_FORCE_LOGO" (layer "B.Cu")
-    (at 189.978572 84.25 180)
+    (at 190.4 89.6 180)
     (attr board_only exclude_from_pos_files exclude_from_bom)
     (fp_text reference "G***" (at 0 0) (layer "B.SilkS") hide
@@
   )
   (footprint "Symbol:KiCad-Logo2_5mm_SilkScreen" (layer "B.Cu")
-    (at 153.8 92.8 180)
+    (at 153.8 96.4 180)
     (descr "KiCad Logo")
     (tags "Logo KiCad")
@@
   )
   (footprint "Symbol:OSHW-Symbol_13.4x12mm_SilkScreen" (layer "B.Cu")
-    (at 153.478572 83.25 180)
+    (at 153.478572 86.85 180)
     (descr "Open Source Hardware Symbol")
     (tags "Logo Symbol OSHW")
@@
   (gr_arc (start 145.4 70) (mid 147.333095 65.333095) (end 152 63.4)
     (stroke (width 0.1) (type default)) (layer "Edge.Cuts"))
-  (gr_text "Super Buttton By FRC 1721 Tidal Force\nhttps://www.frc1721.org/\n${FULL_REVISION}" (at 172.25 101.2) (layer "B.SilkS")
+  (gr_text "By FRC 1721 Tidal Force\nConcord, NH\nhttps://www.frc1721.org/\n${FULL_REVISION}" (at 172.25 101.2) (layer "B.SilkS")
     (effects (font (size 0.9 0.9) (thickness 0.2)) (justify mirror))
   )
@@
     (effects (font (size 1.1 1.1) (thickness 0.275) bold) (justify left bottom mirror))
   )
+  (gr_text "Programmable\nSingle Key \nKeyboard" (at 187.8 66.4) (layer "B.SilkS")
+    (effects (font (size 1 1) (thickness 0.25) bold) (justify left top mirror))
+  )
   (dimension (type aligned) (layer "Dwgs.User")
     (pts (xy 189.6 63.4) (xy 189.6 116.6))
@@
   (via (at 194.5 99.5) (size 0.8) (drill 0.4) (layers "F.Cu" "B.Cu") (free) (net 1))
   (via (at 184.75 78.75) (size 0.8) (drill 0.4) (layers "F.Cu" "B.Cu") (free) (net 1))
-  (via (at 174 74) (size 0.8) (drill 0.4) (layers "F.Cu" "B.Cu") (free) (net 1))
+  (via (at 174.6 75) (size 0.8) (drill 0.4) (layers "F.Cu" "B.Cu") (free) (net 1))
   (via (at 164 102.25) (size 0.8) (drill 0.4) (layers "F.Cu" "B.Cu") (free) (net 1))
   (via (at 194.5 80.75) (size 0.8) (drill 0.4) (layers "F.Cu" "B.Cu") (free) (net 1))
   (via (at 182.25 100.5) (size 0.8) (drill 0.4) (layers "F.Cu" "B.Cu") (free) (net 1))
-  (via (at 169.75 74) (size 0.8) (drill 0.4) (layers "F.Cu" "B.Cu") (free) (net 1))
+  (via (at 169.75 73.342929) (size 0.8) (drill 0.4) (layers "F.Cu" "B.Cu") (free) (net 1))
   (via (at 156.75 77.5) (size 0.8) (drill 0.4) (layers "F.Cu" "B.Cu") (free) (net 1))
   (via (at 165 70.75) (size 0.8) (drill 0.4) (layers "F.Cu" "B.Cu") (free) (net 1))
@@
   (segment (start 181.45 76.75) (end 187.75 76.75) (width 0.6) (layer "F.Cu") (net 2))
   (segment (start 168.75 72.463446) (end 168.770017 72.443429) (width 0.6) (layer "F.Cu") (net 2))
-  (segment (start 191.5875 87.8125) (end 173.978572 105.421428) (width 0.6) (layer "F.Cu") (net 2))
   (segment (start 168.75 72.5) (end 168.75 72.463446) (width 0.6) (layer "F.Cu") (net 2))
   (segment (start 168.75 72.5) (end 169.328572 71.921428) (width 0.6) (layer "F.Cu") (net 2))
@@
   (via (at 168.770017 72.443429) (size 0.8) (drill 0.4) (layers "F.Cu" "B.Cu") (net 2))
   (via (at 174.75 72.5) (size 0.8) (drill 0.4) (layers "F.Cu" "B.Cu") (net 2))
+  (via (at 191.5875 95.25) (size 0.8) (drill 0.4) (layers "F.Cu" "B.Cu") (net 2))
+  (segment (start 191.5875 95.25) (end 189.4375 97.4) (width 0.6) (layer "B.Cu") (net 2))
+  (segment (start 189.4375 97.4) (end 182 97.4) (width 0.6) (layer "B.Cu") (net 2))
   (segment (start 174.693429 72.443429) (end 174.75 72.5) (width 0.6) (layer "B.Cu") (net 2))
   (segment (start 168.770017 72.443429) (end 174.693429 72.443429) (width 0.6) (layer "B.Cu") (net 2))
+  (segment (start 182 97.4) (end 174 105.4) (width 0.6) (layer "B.Cu") (net 2))
   (segment (start 171.75 70) (end 172.25 70) (width 0.23) (layer "F.Cu") (net 3))
   (segment (start 164.737676 76.683708) (end 163.609608 75.55564) (width 0.360923) (layer "F.Cu") (net 3))
@@
   (segment (start 176.145235 76.145235) (end 180.55 80.55) (width 0.6) (layer "F.Cu") (net 12))
   (segment (start 168.37 80.12) (end 168.37 79) (width 0.6) (layer "F.Cu") (net 13))
-  (segment (start 190.5 97.75) (end 191.5875 97.75) (width 0.6) (layer "F.Cu") (net 13))
-  (segment (start 189.5 93.5) (end 189.5 96.75) (width 0.6) (layer "F.Cu") (net 13))
   (segment (start 189.5 96.75) (end 190.5 97.75) (width 0.6) (layer "F.Cu") (net 13))
-  (segment (start 189 93) (end 189.5 93.5) (width 0.6) (layer "F.Cu") (net 13))
   (segment (start 186.25 91.25) (end 175.5 80.5) (width 0.6) (layer "F.Cu") (net 13))
   (segment (start 175.5 80.5) (end 168.75 80.5) (width 0.6) (layer "F.Cu") (net 13))
   (segment (start 168.75 80.5) (end 168.37 80.12) (width 0.6) (layer "F.Cu") (net 13))
-  (via (at 186.25 91.25) (size 0.8) (drill 0.4) (layers "F.Cu" "B.Cu") (net 13))
-  (via (at 189 93) (size 0.8) (drill 0.4) (layers "F.Cu" "B.Cu") (net 13))
-  (segment (start 186.25 91.25) (end 187.75 92.75) (width 0.6) (layer "B.Cu") (net 13))
-  (segment (start 188.75 92.75) (end 189 93) (width 0.6) (layer "B.Cu") (net 13))
-  (segment (start 187.75 92.75) (end 188.75 92.75) (width 0.6) (layer "B.Cu") (net 13))
-  (segment (start 179.75 87.75) (end 179.75 90.75) (width 0.6) (layer "F.Cu") (net 14))
-  (segment (start 179.75 90.75) (end 177.25 93.25) (width 0.6) (layer "F.Cu") (net 14))
-  (segment (start 173.5 81.5) (end 179.75 87.75) (width 0.6) (layer "F.Cu") (net 14))
-  (segment (start 167.1 79.98137) (end 168.61863 81.5) (width 0.6) (layer "F.Cu") (net 14))
-  (segment (start 167.1 79) (end 167.1 79.98137) (width 0.6) (layer "F.Cu") (net 14))
-  (segment (start 175.5 93.25) (end 165.425 103.325) (width 0.6) (layer "F.Cu") (net 14))
-  (segment (start 165.425 103.325) (end 165.425 105.5) (width 0.6) (layer "F.Cu") (net 14))
-  (segment (start 177.25 93.25) (end 175.5 93.25) (width 0.6) (layer "F.Cu") (net 14))
-  (segment (start 168.61863 81.5) (end 173.5 81.5) (width 0.6) (layer "F.Cu") (net 14))
+  (segment (start 190.5 97.75) (end 191.5875 97.75) (width 0.6) (layer "F.Cu") (net 13))
+  (segment (start 186.25 91.25) (end 189.5 94.5) (width 0.6) (layer "F.Cu") (net 13))
+  (segment (start 189.5 94.5) (end 189.5 96.75) (width 0.6) (layer "F.Cu") (net 13))
+  (segment (start 167.97672 80.998807) (end 167.1 80.122087) (width 0.6) (layer "F.Cu") (net 14))
+  (segment (start 167.1 80.122087) (end 167.1 79) (width 0.6) (layer "F.Cu") (net 14))
+  (via (at 167.97672 80.998807) (size 0.8) (drill 0.4) (layers "F.Cu" "B.Cu") (net 14))
+  (via (at 165.425 105.5) (size 0.8) (drill 0.4) (layers "F.Cu" "B.Cu") (net 14))
+  (segment (start 165.4 85.6) (end 165.4 105.475) (width 0.6) (layer "B.Cu") (net 14))
+  (segment (start 167.97672 83.02328) (end 165.4 85.6) (width 0.6) (layer "B.Cu") (net 14))
+  (segment (start 167.97672 80.998807) (end 167.97672 83.02328) (width 0.6) (layer "B.Cu") (net 14))
+  (segment (start 165.4 105.475) (end 165.425 105.5) (width 0.6) (layer "B.Cu") (net 14))
   (segment (start 165.83 80.37) (end 165.8 80.4) (width 0.25) (layer "F.Cu") (net 16))
   (segment (start 165.83 79) (end 165.83 80.37) (width 0.25) (layer "F.Cu") (net 16))
