File: Hardware/SuperButtonX1/SuperButtonX1.kicad_sch (KiCad schematic)
At the start: 21 parts, among them J101 USBC, J103 EXT_LED, SW101 Switch, SW201 PROG, U101 CH552G

Commit message: Include LCSC part numbers in BOM
Parts:
- C101, C104: LCSC# (none) -> C138340
- D103, D104: LCSC# (none) -> C130114
- J101: LCSC# (none) -> C319148
- R101, R102: LCSC# (none) -> C269748
- R103, R104, R105, R106, R108: LCSC# (none) -> C384454
- SW201: LCSC# (none) -> C318884
- U101: LCSC C111292 -> (none); LCSC# (none) -> C111292
Changed lines of the file:
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@@
+      (effects (font (size 1.27 1.27)) hide)
+    )
+    (property "LCSC#" "C384454" (at 242.57 27.305 0)
       (effects (font (size 1.27 1.27)) hide)
     )
@@
       (effects (font (size 1.27 1.27)) hide)
     )
+    (property "LCSC#" "C384454" (at 226.695 33.655 90)
+      (effects (font (size 1.27 1.27)) hide)
+    )
     (pin "1")
     (pin "2")
@@
     )
     (property "Datasheet" "~" (at 175.895 34.29 0)
+      (effects (font (size 1.27 1.27)) hide)
+    )
+    (property "LCSC#" "C318884" (at 175.895 39.37 0)
       (effects (font (size 1.27 1.27)) hide)
     )
@@
       (effects (font (size 1.27 1.27)) hide)
     )
+    (property "LCSC#" "C138340" (at 179.07 22.86 0)
+      (effects (font (size 1.27 1.27)) hide)
+    )
     (pin "1")
     (pin "2")
@@
     )
     (property "Datasheet" "~" (at 57.785 37.465 0)
+      (effects (font (size 1.27 1.27)) hide)
+    )
+    (property "LCSC#" "C269748" (at 57.785 37.465 0)
       (effects (font (size 1.27 1.27)) hide)
     )
@@
       (effects (font (size 1.27 1.27)) hide)
     )
-    (property "LCSC" "C111292" (at 118.745 46.355 0)
+    (property "LCSC#" "C111292" (at 118.745 46.355 0)
       (effects (font (size 1.27 1.27)) hide)
     )
@@
     )
     (property "Datasheet" "https://www.usb.org/sites/default/files/documents/usb_type-c.zip" (at 30.48 41.275 0)
+      (effects (font (size 1.27 1.27)) hide)
+    )
+    (property "LCSC#" "C319148" (at 26.67 41.275 0)
       (effects (font (size 1.27 1.27)) hide)
     )
@@
       (effects (font (size 1.27 1.27)) hide)
     )
+    (property "LCSC#" "C130114" (at 242.57 34.29 90)
+      (effects (font (size 1.27 1.27)) hide)
+    )
     (pin "1")
     (pin "2")
@@
     )
     (property "Datasheet" "~" (at 168.275 22.86 0)
+      (effects (font (size 1.27 1.27)) hide)
+    )
+    (property "LCSC#" "C138340" (at 168.275 22.86 0)
       (effects (font (size 1.27 1.27)) hide)
     )
@@
       (effects (font (size 1.27 1.27)) hide)
     )
+    (property "LCSC#" "C269748" (at 68.58 37.465 0)
+      (effects (font (size 1.27 1.27)) hide)
+    )
     (pin "1")
     (pin "2")
@@
       (effects (font (size 1.27 1.27)) hide)
     )
+    (property "LCSC#" "C384454" (at 166.37 39.37 90)
+      (effects (font (size 1.27 1.27)) hide)
+    )
     (pin "1")
     (pin "2")
@@
     )
     (property "Datasheet" "~" (at 233.68 60.96 0)
+      (effects (font (size 1.27 1.27)) hide)
+    )
+    (property "LCSC#" "C384454" (at 233.68 60.96 90)
       (effects (font (size 1.27 1.27)) hide)
     )
@@
       (effects (font (size 1.27 1.27)) hide)
     )
+    (property "LCSC#" "C384454" (at 255.27 27.305 0)
+      (effects (font (size 1.27 1.27)) hide)
+    )
     (pin "1")
     (pin "2")
@@
       (effects (font (size 1.27 1.27)) hide)
     )
+    (property "LCSC#" "C130114" (at 255.27 34.29 90)
+      (effects (font (size 1.27 1.27)) hide)
+    )

Commit message: Swap out
Parts:
- R103, R104, R105, R106, R108: LCSC# C384454 -> C2889545
Changed lines of the file:
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@@
       (effects (font (size 1.27 1.27)) hide)
     )
-    (property "LCSC#" "C384454" (at 242.57 27.305 0)
+    (property "LCSC#" "C2889545" (at 242.57 27.305 0)
       (effects (font (size 1.27 1.27)) hide)
     )
@@
       (effects (font (size 1.27 1.27)) hide)
     )
-    (property "LCSC#" "C384454" (at 226.695 33.655 90)
+    (property "LCSC#" "C2889545" (at 226.695 33.655 90)
       (effects (font (size 1.27 1.27)) hide)
     )
@@
       (effects (font (size 1.27 1.27)) hide)
     )
-    (property "LCSC#" "C384454" (at 166.37 39.37 90)
+    (property "LCSC#" "C2889545" (at 166.37 39.37 90)
       (effects (font (size 1.27 1.27)) hide)
     )
@@
       (effects (font (size 1.27 1.27)) hide)
     )
-    (property "LCSC#" "C384454" (at 233.68 60.96 90)
+    (property "LCSC#" "C2889545" (at 233.68 60.96 90)
       (effects (font (size 1.27 1.27)) hide)
     )
@@
       (effects (font (size 1.27 1.27)) hide)
     )
-    (property "LCSC#" "C384454" (at 255.27 27.305 0)
-      (effects (font (size 1.27 1.27)) hide)
-    )
+    (property "LCSC#" "C2889545" (at 255.27 27.305 0)
+      (effects (font (size 1.27 1.27)) hide)
+    )

Commit message: Clean up Super Button X1
Parts:
- C101, C104: LCSC# C138340 -> C49678
- D103, D104: LCSC# C130114 -> C84256
- R103, R104, R105, R106, R108: LCSC# C2889545 -> C17606
Changed lines of the file:
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@@
       (effects (font (size 1.27 1.27)) hide)
     )
-    (property "LCSC#" "C2889545" (at 242.57 27.305 0)
+    (property "LCSC#" "C17606" (at 242.57 27.305 0)
       (effects (font (size 1.27 1.27)) hide)
     )
@@
       (effects (font (size 1.27 1.27)) hide)
     )
-    (property "LCSC#" "C2889545" (at 226.695 33.655 90)
+    (property "LCSC#" "C17606" (at 226.695 33.655 90)
       (effects (font (size 1.27 1.27)) hide)
     )
@@
       (effects (font (size 1.27 1.27)) hide)
     )
-    (property "LCSC#" "C138340" (at 179.07 22.86 0)
+    (property "LCSC#" "C49678" (at 179.07 22.86 0)
       (effects (font (size 1.27 1.27)) hide)
     )
@@
       (effects (font (size 1.27 1.27)) hide)
     )
-    (property "LCSC#" "C130114" (at 242.57 34.29 90)
+    (property "LCSC#" "C84256" (at 242.57 34.29 90)
       (effects (font (size 1.27 1.27)) hide)
     )
@@
       (effects (font (size 1.27 1.27)) hide)
     )
-    (property "LCSC#" "C138340" (at 168.275 22.86 0)
+    (property "LCSC#" "C49678" (at 168.275 22.86 0)
       (effects (font (size 1.27 1.27)) hide)
     )
@@
       (effects (font (size 1.27 1.27)) hide)
     )
-    (property "LCSC#" "C2889545" (at 166.37 39.37 90)
+    (property "LCSC#" "C17606" (at 166.37 39.37 90)
       (effects (font (size 1.27 1.27)) hide)
     )
@@
       (effects (font (size 1.27 1.27)) hide)
     )
-    (property "LCSC#" "C2889545" (at 233.68 60.96 90)
+    (property "LCSC#" "C17606" (at 233.68 60.96 90)
       (effects (font (size 1.27 1.27)) hide)
     )
@@
       (effects (font (size 1.27 1.27)) hide)
     )
-    (property "LCSC#" "C2889545" (at 255.27 27.305 0)
+    (property "LCSC#" "C17606" (at 255.27 27.305 0)
       (effects (font (size 1.27 1.27)) hide)
     )
@@
       (effects (font (size 1.27 1.27)) hide)
     )
-    (property "LCSC#" "C130114" (at 255.27 34.29 90)
-      (effects (font (size 1.27 1.27)) hide)
-    )
+    (property "LCSC#" "C84256" (at 255.27 34.29 90)
+      (effects (font (size 1.27 1.27)) hide)
+    )
