File: Hardware/SuperButtonX1/SuperButtonX1.kicad_sch (KiCad schematic)
At the start: 21 parts, among them J101 USBC, J103 EXT_LED, SW101 Switch, SW201 PROG, U101 CH552G

Commit message: Feat/Variants (#4)
Co-authored-by: Jack Jewett <jewett818@gmail.com>
Parts:
- C101, C104: LCSC# (none) -> C49678
- D103, D104: LCSC# (none) -> C84256
- J101: LCSC# (none) -> C319148
- R101, R102: LCSC# (none) -> C269748
- R103, R104, R105, R106, R108: LCSC# (none) -> C17606
- SW201: LCSC# (none) -> C318884
- U101: LCSC C111292 -> (none); LCSC# (none) -> C111292
