File: Hardware/SuperButtonX3/SuperButtonX3.kicad_sch (KiCad schematic)
At the start: 25 parts, among them J101 USBC, J103 EXT_LED, SW101 Switch, SW103 Switch, SW104 Switch, SW201 PROG, U101 CH552G

Commit message: Clean up x3 board
Connections:
- net SW_SENSE2: now also U101.10 (P3.3)
- net SW_SENSE3: now also U101.11 (P3.4)
Changed lines of the file:
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@@
   (no_connect (at 131.445 32.385))
   (no_connect (at 41.91 56.515))
-  (wire (pts (xy 142.875 60.325) (xy 131.445 60.325))
-    (stroke (width 0) (type default))
-  )
   (wire (pts (xy 274.955 26.67) (xy 274.955 27.305))
     (stroke (width 0) (type default))
@@
     (stroke (width 0) (type default))
   )
-  (wire (pts (xy 142.875 55.245) (xy 131.445 55.245))
+  (wire (pts (xy 131.445 55.245) (xy 146.05 55.245))
     (stroke (width 0) (type default))
   )
@@
     (stroke (width 0) (type default))
   )
-  (wire (pts (xy 142.875 47.625) (xy 131.445 47.625))
+  (wire (pts (xy 131.445 47.625) (xy 146.05 47.625))
     (stroke (width 0) (type default))
   )
@@
     (stroke (width 0) (type default))
   )
-  (wire (pts (xy 142.875 57.785) (xy 131.445 57.785))
-    (stroke (width 0) (type default))
-  )
   (wire (pts (xy 211.455 66.675) (xy 211.455 60.96))
     (stroke (width 0) (type default))
   )
-  (wire (pts (xy 142.748 50.165) (xy 131.445 50.165))
-    (stroke (width 0) (type default))
-  )
   (wire (pts (xy 168.275 25.4) (xy 168.275 26.035))
     (stroke (width 0) (type default))
@@
     (stroke (width 0) (type default))
   )
+  (wire (pts (xy 131.445 57.785) (xy 146.05 57.785))
+    (stroke (width 0) (type default))
+  )
   (wire (pts (xy 263.525 62.23) (xy 265.43 62.23))
     (stroke (width 0) (type default))
@@
     (stroke (width 0) (type default))
   )
+  (wire (pts (xy 131.445 60.325) (xy 146.05 60.325))
+    (stroke (width 0) (type default))
+  )
   (wire (pts (xy 19.05 64.135) (xy 19.05 66.04))
     (stroke (width 0) (type default))
@@
     (stroke (width 0) (type default))
   )
+  (wire (pts (xy 131.445 50.165) (xy 146.05 50.165))
+    (stroke (width 0) (type default))
+  )
   (polyline (pts (xy 283.845 13.335) (xy 283.845 74.93))
     (stroke (width 0) (type default))
@@
     (stroke (width 0) (type default))
   )
-  (wire (pts (xy 142.748 52.705) (xy 131.445 52.705))
+  (wire (pts (xy 131.445 52.705) (xy 146.05 52.705))
     (stroke (width 0) (type default))
   )
@@
     (stroke (width 0) (type default))
   )
-  (wire (pts (xy 142.875 45.085) (xy 131.445 45.085))
+  (wire (pts (xy 131.445 45.085) (xy 146.05 45.085))
     (stroke (width 0) (type default))
   )
@@
     (effects (font (size 1.27 1.27)) (justify left bottom))
   )
-  (label "EXT" (at 142.875 57.785 180) (fields_autoplaced)
+  (label "EXT" (at 146.05 57.785 180) (fields_autoplaced)
     (effects (font (size 1.27 1.27)) (justify right bottom))
   )
@@
     (effects (font (size 1.27 1.27)) (justify left bottom))
   )
-  (label "SW_SENSE3" (at 132.08 50.292 0) (fields_autoplaced)
-    (effects (font (size 1.27 1.27)) (justify left bottom))
+  (label "SW_SENSE3" (at 146.05 50.165 180) (fields_autoplaced)
+    (effects (font (size 1.27 1.27)) (justify right bottom))
   )
   (label "USB+" (at 48.895 43.815 180) (fields_autoplaced)
     (effects (font (size 1.27 1.27)) (justify right bottom))
   )
-  (label "USB-" (at 142.875 45.085 180) (fields_autoplaced)
+  (label "USB-" (at 146.05 45.085 180) (fields_autoplaced)
     (effects (font (size 1.27 1.27)) (justify right bottom))
   )
@@
     (effects (font (size 1.27 1.27)) (justify right bottom))
   )
-  (label "SW_SENSE1" (at 142.875 55.245 180) (fields_autoplaced)
+  (label "SW_SENSE1" (at 146.05 55.245 180) (fields_autoplaced)
     (effects (font (size 1.27 1.27)) (justify right bottom))
   )
@@
     (effects (font (size 1.27 1.27)) (justify right bottom))
   )
-  (label "STAT" (at 142.875 60.325 180) (fields_autoplaced)
-    (effects (font (size 1.27 1.27)) (justify right bottom))
-  )
-  (label "USB+" (at 142.875 47.625 180) (fields_autoplaced)
+  (label "STAT" (at 146.05 60.325 180) (fields_autoplaced)
+    (effects (font (size 1.27 1.27)) (justify right bottom))
+  )
+  (label "USB+" (at 146.05 47.625 180) (fields_autoplaced)
     (effects (font (size 1.27 1.27)) (justify right bottom))
   )
@@
     (effects (font (size 1.27 1.27)) (justify left bottom))
   )
-  (label "SW_SENSE2" (at 132.08 52.832 0) (fields_autoplaced)
-    (effects (font (size 1.27 1.27)) (justify left bottom))
+  (label "SW_SENSE2" (at 146.05 52.705 180) (fields_autoplaced)
+    (effects (font (size 1.27 1.27)) (justify right bottom))
   )
   (label "USB+" (at 156.845 39.37 0) (fields_autoplaced)

Commit message: Fix routing
Connections:
- net SW_SENSE2: now also U101.2 (P1.4); no longer U101.10 (P3.3)
- net SW_SENSE3: now also U101.3 (P1.5); no longer U101.11 (P3.4)
Changed lines of the file:
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@@
   (junction (at 22.86 66.04) (diameter 0) (color 0 0 0 0)
   )
-  (no_connect (at 131.445 37.465))
-  (no_connect (at 131.445 34.925))
+  (no_connect (at 131.445 52.705))
   (no_connect (at 131.445 40.005))
   (no_connect (at 41.91 53.975))
@@
   (no_connect (at 131.445 32.385))
   (no_connect (at 41.91 56.515))
+  (no_connect (at 131.445 50.165))
   (wire (pts (xy 274.955 26.67) (xy 274.955 27.305))
     (stroke (width 0) (type default))
@@
     (stroke (width 0) (type default))
   )
+  (wire (pts (xy 131.445 37.465) (xy 146.05 37.465))
+    (stroke (width 0) (type default))
+  )
   (wire (pts (xy 41.91 33.655) (xy 57.785 33.655))
     (stroke (width 0) (type default))
@@
     (stroke (width 0) (type default))
   )
-  (wire (pts (xy 131.445 50.165) (xy 146.05 50.165))
+  (wire (pts (xy 131.445 34.925) (xy 146.05 34.925))
     (stroke (width 0) (type default))
   )
@@
     (stroke (width 0) (type default))
   )
-  (wire (pts (xy 131.445 52.705) (xy 146.05 52.705))
-    (stroke (width 0) (type default))
-  )
   (wire (pts (xy 68.58 31.115) (xy 68.58 34.925))
     (stroke (width 0) (type default))
@@
     (effects (font (size 1.27 1.27)) (justify left bottom))
   )
-  (label "SW_SENSE3" (at 146.05 50.165 180) (fields_autoplaced)
+  (label "SW_SENSE3" (at 146.05 34.925 180) (fields_autoplaced)
     (effects (font (size 1.27 1.27)) (justify right bottom))
   )
@@
     (effects (font (size 1.27 1.27)) (justify left bottom))
   )
-  (label "SW_SENSE2" (at 146.05 52.705 180) (fields_autoplaced)
-    (effects (font (size 1.27 1.27)) (justify right bottom))
-  )
+  (label "SW_SENSE2" (at 146.05 37.465 180) (fields_autoplaced)
+    (effects (font (size 1.27 1.27)) (justify right bottom))
+  )
